Commit message: 20260405 加入apriltag urdf的FK经过仿射校正后准确,手眼标定尚不准确

File: SO101/so101_5dof_stylus_2.urdf (robot description, URDF)
Before this commit: robot so101_old_calib, 7 links, 6 joints
Links:
- removed link base
- removed link gripper
- removed link jaw
- removed link lower_arm
- removed link shoulder
- removed link upper_arm
- removed link wrist
- added link base_link, mass 0.147; collision mesh filename=assets/base_motor_holder_so101_v1.stl; collision mesh filename=assets/base_so101_v2.stl
- added link end_effector_stylus_link, mass 0.020; collision mesh filename=assets/pen_cap.stl; collision mesh filename=assets/trans_board.stl
- added link lower_arm_link, mass 0.104; collision mesh filename=assets/motor_holder_so101_wrist_v1.stl; collision mesh filename=assets/sts3215_03a_v1.stl
- added link shoulder_link, mass 0.100006; collision mesh filename=assets/motor_holder_so101_base_v1.stl; collision mesh filename=assets/rotation_pitch_so101_v1.stl
- added link stylus_tcp_link, mass 1e-9
- added link upper_arm_link, mass 0.103; collision mesh filename=assets/sts3215_03a_v1.stl; collision mesh filename=assets/upper_arm_so101_v1.stl
- added link wrist_link, mass 0.079; collision mesh filename=assets/sts3215_03a_no_horn_v1.stl; collision mesh filename=assets/wrist_roll_pitch_so101_v2.stl
Joints:
- removed joint gripper
- added joint stylus_tcp_joint: type fixed, parent end_effector_stylus_link, child stylus_tcp_link, origin xyz=0 0 -0.095 rpy=0 0 0, axis 0 0 0
- joint elbow_flex: child lower_arm -> lower_arm_link; limit lower=-0.174533 upper=3.14159 effort=10 velocity=10 -> lower=-1.69 upper=1.69 effort=10 velocity=10; origin xyz=-0.028 0.11257 1.24466e-16 rpy=1.89432e-15 -3.22659e-15 -3.14159 -> xyz=-0.11257 -0.028 1.73763e-16 rpy=-3.63608e-16 8.74301e-16 1.5708; parent upper_arm -> upper_arm_link
- joint shoulder_lift: child upper_arm -> upper_arm_link; limit lower=-3.31613 upper=0.174533 effort=10 velocity=10 -> lower=-1.74533 upper=1.74533 effort=10 velocity=10; origin xyz=-0.0303992 -0.0182778 -0.0542 rpy=-1.5708 1.5708 0 -> xyz=-0.0303992 -0.0182778 -0.0542 rpy=-1.5708 -1.5708 0; parent shoulder -> shoulder_link
- joint shoulder_pan: child shoulder -> shoulder_link; origin xyz=0.0207909 -0.0230745 0.0948817 rpy=-3.14159 6.03684e-16 1.5708 -> xyz=0.0388353 -8.97657e-09 0.0624 rpy=3.14159 4.18253e-17 -3.14159; parent base -> base_link
- joint wrist_flex: child wrist -> wrist_link; origin xyz=-0.0052 -0.1349 3.40439e-16 rpy=-1.41553e-15 4.91611e-15 7.56157e-09 -> xyz=-0.1349 0.0052 3.62355e-17 rpy=4.02456e-15 8.67362e-16 -1.5708; parent lower_arm -> lower_arm_link
- joint wrist_roll: child gripper -> end_effector_stylus_link; limit lower=-2.79253 upper=2.79253 effort=10 velocity=10 -> lower=-2.74385 upper=2.84121 effort=10 velocity=10; origin xyz=2.77556e-17 -0.0611 0.0181 rpy=1.5708 -9.38083e-08 3.14159 -> xyz=5.55112e-17 -0.0611 0.0181 rpy=1.5708 0.0486795 3.14159; parent wrist -> wrist_link
